File: pcb/ePaper_Display.kicad_sch (KiCad schematic)
At the start: 24 parts, among them Q4 SI1308EDL-T1-GE3

Commit message: switch epaper capacitor to 0402
Parts:
- C12, C16, C17, C18: footprint Capacitor_SMD:C_0603_1608Metric -> Capacitor_SMD:C_0402_1005Metric; LCSC Part C15849 -> C1518208
- C13, C14, C15, C19, C20, C21, C22, C23: footprint Capacitor_SMD:C_0805_2012Metric -> Capacitor_SMD:C_0402_1005Metric; LCSC Part C98192 -> C2858031
Changed lines of the file:
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@@
 			)
 		)
-		(property "Footprint" "Capacitor_SMD:C_0805_2012Metric"
+		(property "Footprint" "Capacitor_SMD:C_0402_1005Metric"
 			(at 103.1748 73.66 0)
 			(effects
@@
 			)
 		)
-		(property "LCSC Part" "C98192"
+		(property "LCSC Part" "C2858031"
 			(at 104.14 77.47 0)
 			(effects
@@
 			)
 		)
-		(property "Footprint" "Capacitor_SMD:C_0603_1608Metric"
+		(property "Footprint" "Capacitor_SMD:C_0402_1005Metric"
 			(at 176.53 105.1052 0)
 			(effects
@@
 			)
 		)
-		(property "LCSC Part" "C15849"
+		(property "LCSC Part" "C1518208"
 			(at 180.34 104.14 0)
 			(effects
@@
 			)
 		)
-		(property "Footprint" "Capacitor_SMD:C_0603_1608Metric"
+		(property "Footprint" "Capacitor_SMD:C_0402_1005Metric"
 			(at 182.88 102.5652 0)
 			(effects
@@
 			)
 		)
-		(property "LCSC Part" "C15849"
+		(property "LCSC Part" "C1518208"
 			(at 186.69 101.6 0)
 			(effects
@@
 			)
 		)
-		(property "Footprint" "Capacitor_SMD:C_0603_1608Metric"
+		(property "Footprint" "Capacitor_SMD:C_0402_1005Metric"
 			(at 170.18 97.4852 0)
 			(effects
@@
 			)
 		)
-		(property "LCSC Part" "C15849"
+		(property "LCSC Part" "C1518208"
 			(at 173.99 96.52 0)
 			(effects
@@
 			)
 		)
-		(property "Footprint" "Capacitor_SMD:C_0805_2012Metric"
+		(property "Footprint" "Capacitor_SMD:C_0402_1005Metric"
 			(at 182.88 112.7252 0)
 			(effects
@@
 			)
 		)
-		(property "LCSC Part" "C98192"
+		(property "LCSC Part" "C2858031"
 			(at 186.69 111.76 0)
 			(effects
@@
 			)
 		)
-		(property "Footprint" "Capacitor_SMD:C_0805_2012Metric"
+		(property "Footprint" "Capacitor_SMD:C_0402_1005Metric"
 			(at 170.18 69.5452 0)
 			(effects
@@
 			)
 		)
-		(property "LCSC Part" "C98192"
+		(property "LCSC Part" "C2858031"
 			(at 173.99 68.58 0)
 			(effects
@@
 			)
 		)
-		(property "Footprint" "Capacitor_SMD:C_0805_2012Metric"
+		(property "Footprint" "Capacitor_SMD:C_0402_1005Metric"
 			(at 176.53 67.0052 0)
 			(effects
@@
 			)
 		)
-		(property "LCSC Part" "C98192"
+		(property "LCSC Part" "C2858031"
 			(at 180.34 66.04 0)
 			(effects
@@
 			)
 		)
-		(property "Footprint" "Capacitor_SMD:C_0805_2012Metric"
+		(property "Footprint" "Capacitor_SMD:C_0402_1005Metric"
 			(at 176.53 115.2652 0)
 			(effects
@@
 			)
 		)
-		(property "LCSC Part" "C98192"
+		(property "LCSC Part" "C2858031"
 			(at 180.34 114.3 0)
 			(effects
@@
 			)
 		)
-		(property "Footprint" "Capacitor_SMD:C_0805_2012Metric"
+		(property "Footprint" "Capacitor_SMD:C_0402_1005Metric"
 			(at 118.4148 90.17 0)
 			(effects
@@
 			)
 		)
-		(property "LCSC Part" "C98192"
+		(property "LCSC Part" "C2858031"
 			(at 119.38 93.98 0)
 			(effects
@@
 			)
 		)
-		(property "Footprint" "Capacitor_SMD:C_0603_1608Metric"
+		(property "Footprint" "Capacitor_SMD:C_0402_1005Metric"
 			(at 170.18 117.8052 0)
 			(effects
@@
 			)
 		)
-		(property "LCSC Part" "C15849"
+		(property "LCSC Part" "C1518208"
 			(at 173.99 116.84 0)
 			(effects
@@
 			)
 		)
-		(property "Footprint" "Capacitor_SMD:C_0805_2012Metric"
+		(property "Footprint" "Capacitor_SMD:C_0402_1005Metric"
 			(at 82.2452 88.9 0)
 			(effects
@@
 			)
 		)
-		(property "LCSC Part" "C98192"
+		(property "LCSC Part" "C2858031"
 			(at 81.28 92.71 0)
 			(effects
@@
 			)
 		)
-		(property "Footprint" "Capacitor_SMD:C_0805_2012Metric"
+		(property "Footprint" "Capacitor_SMD:C_0402_1005Metric"
 			(at 170.18 107.6452 0)
 			(effects
@@
 			)
 		)
-		(property "LCSC Part" "C98192"
+		(property "LCSC Part" "C2858031"
 			(at 173.99 106.68 0)
 			(effects
